File: module_sim800c.sch (KiCad schematic (older format))
At the start: 16 parts, among them J4 SIM_Card, J5 ANTEN, J7 CONN_01X04, SW1 SW_Push, U3 SIM800C-RESCUE-esp32-gateway-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, U8 SP1001

Commit message: edit schematic
Other:
- note added: "MODULE SIM800C"
- moved on the sheet: C5, C6, C8, D3, D4, J4, J5, J7, R12, R13, R14, R17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

Commit message: add footprint mcp1727
Parts:
- D4: footprint LEDs:LED_0603 -> LEDs:LED_D3.0mm
- J5: footprint Pin_Headers:Pin_Header_Straight_1x02_Pitch1.00mm -> footprint:SMA_Straight
- J7: footprint Pin_Headers:Pin_Header_Angled_1x04_Pitch1.27mm -> Pin_Headers:Pin_Header_Straight_1x04_Pitch2.54mm
Changed lines of the file:
@@
 EESchema Schematic File Version 2
+LIBS:PJ-102A
 LIBS:esp32-gateway-hw-rescue
 LIBS:power
@@
 LIBS:sim_card_holder
 LIBS:sp1001
+LIBS:MCP1727-3302E_SN
+LIBS:mcp1727
 LIBS:esp32-gateway-hw-cache
 EELAYER 25 0
@@
 NoConn ~ 6550 4550
 $Comp
-L GND #PWR017
+L GND #PWR21
 U 1 1 59DC6183
 P 6950 5300
-F 0 "#PWR017" H 6950 5050 50  0001 C CNN
+F 0 "#PWR21" H 6950 5050 50  0001 C CNN
 F 1 "GND" H 6950 5150 50  0000 C CNN
 F 2 "" H 6950 5300 50  0001 C CNN
@@
 $EndComp
 $Comp
-L GND #PWR018
+L GND #PWR18
 U 1 1 59DC6189
 P 4050 5050
-F 0 "#PWR018" H 4050 4800 50  0001 C CNN
+F 0 "#PWR18" H 4050 4800 50  0001 C CNN
 F 1 "GND" H 4050 4900 50  0000 C CNN
 F 2 "" H 4050 5050 50  0001 C CNN
@@
 F 0 "J5" H 3500 4950 50  0000 C CNN
 F 1 "ANTEN" H 3500 4550 50  0000 C CNN
-F 2 "Pin_Headers:Pin_Header_Straight_1x02_Pitch1.00mm" H 3500 4750 50  0001 C CNN
+F 2 "footprint:SMA_Straight" H 3500 4750 50  0001 C CNN
 F 3 "" H 3500 4750 50  0001 C CNN
 	1    3500 4750
@@
 F 0 "D4" H 7150 5050 50  0000 C CNN
 F 1 "LED" H 7150 4850 50  0000 C CNN
-F 2 "LEDs:LED_0603" H 7150 4950 50  0001 C CNN
+F 2 "LEDs:LED_D3.0mm" H 7150 4950 50  0001 C CNN
 F 3 "" H 7150 4950 50  0001 C CNN
 	1    7150 4950
@@
 F 0 "J7" H 4450 4250 50  0000 C CNN
 F 1 "CONN_01X04" V 4550 4000 50  0000 C CNN
-F 2 "Pin_Headers:Pin_Header_Angled_1x04_Pitch1.27mm" H 4450 4000 50  0001 C CNN
+F 2 "Pin_Headers:Pin_Header_Straight_1x04_Pitch2.54mm" H 4450 4000 50  0001 C CNN
 F 3 "" H 4450 4000 50  0001 C CNN
 	1    4450 4000
@@
 $EndComp
 $Comp
-L +3V3 #PWR019
+L +3V3 #PWR20
 U 1 1 59DCE5F6
 P 6750 2600
-F 0 "#PWR019" H 6750 2450 50  0001 C CNN
+F 0 "#PWR20" H 6750 2450 50  0001 C CNN
 F 1 "+3V3" H 6750 2740 50  0000 C CNN
 F 2 "" H 6750 2600 50  0001 C CNN
@@
 $EndComp
 $Comp
-L GND #PWR020
+L GND #PWR24
 U 1 1 59DCFA55
 P 7400 4950
-F 0 "#PWR020" H 7400 4700 50  0001 C CNN
+F 0 "#PWR24" H 7400 4700 50  0001 C CNN
 F 1 "GND" H 7400 4800 50  0000 C CNN
 F 2 "" H 7400 4950 50  0001 C CNN
@@
 $EndComp
 $Comp
-L GND #PWR021
+L GND #PWR17
 U 1 1 59DD0AE0
 P 3550 3700
-F 0 "#PWR021" H 3550 3450 50  0001 C CNN
+F 0 "#PWR17" H 3550 3450 50  0001 C CNN
 F 1 "GND" H 3550 3550 50  0000 C CNN
 F 2 "" H 3550 3700 50  0001 C CNN
@@
 $EndComp
 $Comp
-L GND #PWR022
+L GND #PWR19
 U 1 1 59DD0B6C
 P 4150 4050
-F 0 "#PWR022" H 4150 3800 50  0001 C CNN
+F 0 "#PWR19" H 4150 3800 50  0001 C CNN
 F 1 "GND" H 4150 3900 50  0000 C CNN
 F 2 "" H 4150 4050 50  0001 C CNN
@@
 $EndComp
 $Comp
-L GND #PWR023
+L GND #PWR23
 U 1 1 59DD114F
 P 7300 4650
-F 0 "#PWR023" H 7300 4400 50  0001 C CNN
+F 0 "#PWR23" H 7300 4400 50  0001 C CNN
 F 1 "GND" H 7300 4500 50  0000 C CNN
 F 2 "" H 7300 4650 50  0001 C CNN
@@
 $EndComp
 $Comp
-L GND #PWR024
+L GND #PWR25
 U 1 1 59DD1317
 P 7550 3700
-F 0 "#PWR024" H 7550 3450 50  0001 C CNN
+F 0 "#PWR25" H 7550 3450 50  0001 C CNN
 F 1 "GND" H 7550 3550 50  0000 C CNN
 F 2 "" H 7550 3700 50  0001 C CNN
@@
 Connection ~ 6950 3350
 $Comp
-L GND #PWR025
+L GND #PWR22
 U 1 1 59DD1C11
 P 7150 3000
-F 0 "#PWR025" H 7150 2750 50  0001 C CNN
+F 0 "#PWR22" H 7150 2750 50  0001 C CNN
 F 1 "GND" H 7150 2850 50  0000 C CNN
 F 2 "" H 7150 3000 50  0001 C CNN
@@
 GND
 $Comp
-L GND #PWR026
+L GND #PWR27
 U 1 1 59DE63CF
 P 8200 2050
-F 0 "#PWR026" H 8200 1800 50  0001 C CNN
+F 0 "#PWR27" H 8200 1800 50  0001 C CNN
 F 1 "GND" H 8200 1900 50  0000 C CNN
 F 2 "" H 8200 2050 50  0001 C CNN
@@
 $EndComp
 $Comp
-L +3.3V #PWR027
+L +3.3V #PWR26
 U 1 1 59DE6403
 P 8200 1650
-F 0 "#PWR027" H 8200 1500 50  0001 C CNN
+F 0 "#PWR26" H 8200 1500 50  0001 C CNN
 F 1 "+3.3V" H 8200 1790 50  0000 C CNN
 F 2 "" H 8200 1650 50  0001 C CNN

Commit message: edit layout
Parts:
- added C10: 10uF, footprint:C_0603, symbol C
- added C11: 100nF, footprint:C_0603, symbol C
Connections:
- net +3V3: now also C10.2, C11.2
- net GND: now also C10.1, C11.1
Changed lines of the file:
@@
 LIBS:sim_card_holder
 LIBS:sp1001
-LIBS:MCP1727-3302E_SN
 LIBS:mcp1727
 LIBS:esp32-gateway-hw-cache
@@
 NoConn ~ 6550 4550
 $Comp
-L GND #PWR21
+L GND #PWR017
 U 1 1 59DC6183
 P 6950 5300
-F 0 "#PWR21" H 6950 5050 50  0001 C CNN
+F 0 "#PWR017" H 6950 5050 50  0001 C CNN
 F 1 "GND" H 6950 5150 50  0000 C CNN
 F 2 "" H 6950 5300 50  0001 C CNN
@@
 $EndComp
 $Comp
-L GND #PWR18
+L GND #PWR018
 U 1 1 59DC6189
 P 4050 5050
-F 0 "#PWR18" H 4050 4800 50  0001 C CNN
+F 0 "#PWR018" H 4050 4800 50  0001 C CNN
 F 1 "GND" H 4050 4900 50  0000 C CNN
 F 2 "" H 4050 5050 50  0001 C CNN
@@
 $EndComp
 $Comp
-L +3V3 #PWR20
+L +3V3 #PWR019
 U 1 1 59DCE5F6
 P 6750 2600
-F 0 "#PWR20" H 6750 2450 50  0001 C CNN
+F 0 "#PWR019" H 6750 2450 50  0001 C CNN
 F 1 "+3V3" H 6750 2740 50  0000 C CNN
 F 2 "" H 6750 2600 50  0001 C CNN
@@
 $EndComp
 $Comp
-L GND #PWR24
+L GND #PWR020
 U 1 1 59DCFA55
 P 7400 4950
-F 0 "#PWR24" H 7400 4700 50  0001 C CNN
+F 0 "#PWR020" H 7400 4700 50  0001 C CNN
 F 1 "GND" H 7400 4800 50  0000 C CNN
 F 2 "" H 7400 4950 50  0001 C CNN
@@
 $EndComp
 $Comp
-L GND #PWR17
+L GND #PWR021
 U 1 1 59DD0AE0
 P 3550 3700
-F 0 "#PWR17" H 3550 3450 50  0001 C CNN
+F 0 "#PWR021" H 3550 3450 50  0001 C CNN
 F 1 "GND" H 3550 3550 50  0000 C CNN
 F 2 "" H 3550 3700 50  0001 C CNN
@@
 $EndComp
 $Comp
-L GND #PWR19
+L GND #PWR022
 U 1 1 59DD0B6C
 P 4150 4050
-F 0 "#PWR19" H 4150 3800 50  0001 C CNN
+F 0 "#PWR022" H 4150 3800 50  0001 C CNN
 F 1 "GND" H 4150 3900 50  0000 C CNN
 F 2 "" H 4150 4050 50  0001 C CNN
@@
 $EndComp
 $Comp
-L GND #PWR23
+L GND #PWR023
 U 1 1 59DD114F
 P 7300 4650
-F 0 "#PWR23" H 7300 4400 50  0001 C CNN
+F 0 "#PWR023" H 7300 4400 50  0001 C CNN
 F 1 "GND" H 7300 4500 50  0000 C CNN
 F 2 "" H 7300 4650 50  0001 C CNN
@@
 $EndComp
 $Comp
-L GND #PWR25
+L GND #PWR024
 U 1 1 59DD1317
 P 7550 3700
-F 0 "#PWR25" H 7550 3450 50  0001 C CNN
+F 0 "#PWR024" H 7550 3450 50  0001 C CNN
 F 1 "GND" H 7550 3550 50  0000 C CNN
 F 2 "" H 7550 3700 50  0001 C CNN
@@
 Connection ~ 6950 3350
 $Comp
-L GND #PWR22
+L GND #PWR025
 U 1 1 59DD1C11
 P 7150 3000
-F 0 "#PWR22" H 7150 2750 50  0001 C CNN
+F 0 "#PWR025" H 7150 2750 50  0001 C CNN
 F 1 "GND" H 7150 2850 50  0000 C CNN
 F 2 "" H 7150 3000 50  0001 C CNN
@@
 GND
 $Comp
-L GND #PWR27
+L GND #PWR026
 U 1 1 59DE63CF
 P 8200 2050
-F 0 "#PWR27" H 8200 1800 50  0001 C CNN
+F 0 "#PWR026" H 8200 1800 50  0001 C CNN
 F 1 "GND" H 8200 1900 50  0000 C CNN
 F 2 "" H 8200 2050 50  0001 C CNN
@@
 $EndComp
 $Comp
-L +3.3V #PWR26
+L +3.3V #PWR027
 U 1 1 59DE6403
 P 8200 1650
-F 0 "#PWR26" H 8200 1500 50  0001 C CNN
+F 0 "#PWR027" H 8200 1500 50  0001 C CNN
 F 1 "+3.3V" H 8200 1790 50  0000 C CNN
 F 2 "" H 8200 1650 50  0001 C CNN
@@
 Text Notes 4500 1550 0    197  ~ 39
 MODULE SIM800C
+$Comp
+L C C10
+U 1 1 59E5EF68
+P 9200 3250
+F 0 "C10" V 9150 3300 50  0000 L CNN
+F 1 "10uF" V 9050 3150 50  0000 L CNN
+F 2 "footprint:C_0603" H 9238 3100 50  0001 C CNN
+F 3 "" H 9200 3250 50  0001 C CNN
+	1    9200 3250
+	-1   0    0    1
+$EndComp
+$Comp
+L C C11
+U 1 1 59E5EF6F
+P 9550 3250
+F 0 "C11" V 9500 3300 50  0000 L CNN
+F 1 "100nF" V 9400 3150 50  0000 L CNN
+F 2 "footprint:C_0603" H 9588 3100 50  0001 C CNN
+F 3 "" H 9550 3250 50  0001 C CNN
+	1    9550 3250
+	-1   0    0    1
+$EndComp
+Wire Wire Line
+	9200 3100 9200 3050
+Wire Wire Line
+	9200 3050 9550 3050
+Wire Wire Line
+	9550 3050 9550 3100
+Wire Wire Line
+	9200 3400 9200 3500
+Wire Wire Line
+	9200 3500 9550 3500
+Wire Wire Line
+	9550 3500 9550 3400
+$Comp
+L GND #PWR028
+U 1 1 59E5EF7C
+P 9400 3550
+F 0 "#PWR028" H 9400 3300 50  0001 C CNN
+F 1 "GND" H 9400 3400 50  0000 C CNN
+F 2 "" H 9400 3550 50  0001 C CNN
+F 3 "" H 9400 3550 50  0001 C CNN
+	1    9400 3550
+	1    0    0    -1
+$EndComp
+$Comp
+L +3V3 #PWR029
+U 1 1 59E5EF82
+P 9400 2900
+F 0 "#PWR029" H 9400 2750 50  0001 C CNN
+F 1 "+3V3" H 9400 3040 50  0000 C CNN
+F 2 "" H 9400 2900 50  0001 C CNN
+F 3 "" H 9400 2900 50  0001 C CNN
+	1    9400 2900
+	1    0    0    -1
+$EndComp
+Wire Wire Line
+	9400 2900 9400 3050
+Connection ~ 9400 3050
+Wire Wire Line
+	9400 3550 9400 3500
+Connection ~ 9400 3500
 $EndSCHEMATC
